Commit message: add cup

File: src/cup.urdf (robot description, URDF)
Before this commit: robot sink, 1 links, 0 joints
Links:
- removed link base_link
- added link baseLink, mass .1; collision mesh filename=Cup/cup_vhacd.obj scale=0.5 0.5 0.5; visual mesh filename=Cup/textured-0008192.obj scale=0.5 0.5 0.5
