Commit message: save changes

File: src/cup/cup_small.urdf (robot description, URDF)
Before this commit: robot cube.urdf, 1 links, 0 joints
Links:
- link baseLink: geometry collision mesh filename=cup/Cup/cup_vhacd.obj scale=0.5 0.5 0.5; visual mesh filename=cup/Cup/textured-0008192.obj scale=0.5 0.5 0.5
